Commit message: [KMJ] Update: decription package

File: robot/description/urdf/robot.urdf.xacro (robot description, xacro)
@@ -1,26 +1,15 @@
 <?xml version="1.0"?>
-<robot name="my_robot" xmlns:xacro="http://www.ros.org/wiki/xacro">
-  <!-- ===================== -->
-  <!-- Basic parameters      -->
-  <!-- ===================== -->
+<robot name="hospital_delivery_robot" xmlns:xacro="http://www.ros.org/wiki/xacro">
   <xacro:property name="body_length" value="0.8"/>
-  <xacro:property name="body_width"  value="0.59"/>
+  <xacro:property name="body_width" value="0.59"/>
   <xacro:property name="body_height" value="0.19"/>
   <xacro:property name="wheel_separation" value="0.38"/>
-  <xacro:property name="wheel_radius" value="0.0625"/>
-  <xacro:property name="wheel_thickness" value="0.04"/>
-  <xacro:property name="caster_radius" value="0.051"/>
-  <xacro:property name="caster_thickness" value="0.03"/>
-  <!-- mesh file -->
-  <xacro:property name="body_mesh_file" value="package://description/meshes/mesh.stl"/>
-  <xacro:property name="body_mesh_scale" value="1 1 1"/>
-  <!-- mesh origin correction -->
-  <xacro:property name="body_mesh_x" value="0.0"/>
-  <xacro:property name="body_mesh_y" value="0.0"/>
-  <xacro:property name="body_mesh_z" value="0.0"/>
-  <xacro:property name="body_mesh_roll" value="0.0"/>
-  <xacro:property name="body_mesh_pitch" value="0.0"/>
-  <xacro:property name="body_mesh_yaw" value="0.0"/>
-  <!-- ROS-converted sensor positions -->
+  <xacro:property name="drive_wheel_diameter" value="0.125"/>
+  <xacro:property name="drive_wheel_radius" value="0.0625"/>
+  <xacro:property name="drive_wheel_thickness" value="0.04"/>
+  <xacro:property name="lidar_size" value="0.037 0.037 0.024"/>
+  <xacro:property name="imu_size" value="0.045 0.035 0.018"/>
+  <xacro:property name="tof_size" value="0.035 0.02 0.02"/>
+  <xacro:property name="tof_direction_size" value="0.08 0.008 0.008"/>
   <xacro:property name="lidar_x" value="0.27"/>
   <xacro:property name="lidar_y" value="0.0"/>
@@ -29,54 +18,55 @@
   <xacro:property name="imu_y" value="0.0"/>
   <xacro:property name="imu_z" value="0.0"/>
-  <xacro:property name="tof0_x" value="0.22"/>
-  <xacro:property name="tof0_y" value="0.32"/>
-  <xacro:property name="tof0_z" value="0.15"/>
-  <xacro:property name="tof1_x" value="0.22"/>
-  <xacro:property name="tof1_y" value="-0.32"/>
-  <xacro:property name="tof1_z" value="0.15"/>
-  <xacro:property name="tof2_x" value="-0.55"/>
-  <xacro:property name="tof2_y" value="0.28"/>
-  <xacro:property name="tof2_z" value="0.15"/>
-  <xacro:property name="tof3_x" value="-0.55"/>
-  <xacro:property name="tof3_y" value="-0.28"/>
-  <xacro:property name="tof3_z" value="0.15"/>
-  <!-- ===================== -->
-  <!-- Materials             -->
-  <!-- ===================== -->
-  <material name="gray">
-    <color rgba="0.6 0.6 0.6 1.0"/>
+  <xacro:property name="tof_front_left_x" value="0.22"/>
+  <xacro:property name="tof_front_left_y" value="0.32"/>
+  <xacro:property name="tof_front_left_z" value="0.15"/>
+  <xacro:property name="tof_front_left_yaw" value="0.436332"/>
+  <xacro:property name="tof_front_right_x" value="0.22"/>
+  <xacro:property name="tof_front_right_y" value="-0.32"/>
+  <xacro:property name="tof_front_right_z" value="0.15"/>
+  <xacro:property name="tof_front_right_yaw" value="-0.436332"/>
+  <xacro:property name="tof_rear_left_x" value="-0.55"/>
+  <xacro:property name="tof_rear_left_y" value="0.28"/>
+  <xacro:property name="tof_rear_left_z" value="0.15"/>
+  <xacro:property name="tof_rear_left_yaw" value="2.70526"/>
+  <xacro:property name="tof_rear_right_x" value="-0.55"/>
+  <xacro:property name="tof_rear_right_y" value="-0.28"/>
+  <xacro:property name="tof_rear_right_z" value="0.15"/>
+  <xacro:property name="tof_rear_right_yaw" value="-2.70526"/>
+  <material name="body_gray">
+    <color rgba="0.55 0.58 0.62 1.0"/>
   </material>
-  <material name="black">
-    <color rgba="0.1 0.1 0.1 1.0"/>
+  <material name="wheel_black">
+    <color rgba="0.04 0.04 0.04 1.0"/>
   </material>
-  <material name="blue">
-    <color rgba="0.2 0.4 1.0 1.0"/>
+  <material name="lidar_blue">
+    <color rgba="0.1 0.35 0.95 1.0"/>
   </material>
-  <material name="green">
-    <color rgba="0.2 0.8 0.2 1.0"/>
+  <material name="imu_green">
+    <color rgba="0.0 0.65 0.25 1.0"/>
   </material>
-  <!-- ===================== -->
-  <!-- base_footprint        -->
-  <!-- ===================== -->
+  <material name="tof_orange">
+    <color rgba="1.0 0.45 0.05 1.0"/>
+  </material>
+  <material name="tof_direction_yellow">
+    <color rgba="1.0 0.9 0.1 1.0"/>
+  </material>
   <link name="base_footprint"/>
   <joint name="base_footprint_to_base_link" type="fixed">
     <parent link="base_footprint"/>
     <child link="base_link"/>
-    <origin xyz="0 0 ${wheel_radius}" rpy="0 0 0"/>
+    <origin xyz="0 0 ${drive_wheel_radius}" rpy="0 0 0"/>
   </joint>
-  <!-- ===================== -->
-  <!-- base_link             -->
-  <!-- ===================== -->
   <link name="base_link">
+    <!-- TODO: Replace body primitive with Fusion 360 STL or DAE mesh after export. -->
     <visual>
-      <origin xyz="${body_mesh_x} ${body_mesh_y} ${body_mesh_z}"
-              rpy="${body_mesh_roll} ${body_mesh_pitch} ${body_mesh_yaw}"/>
+      <origin xyz="0 0 ${body_height / 2.0 - drive_wheel_radius}" rpy="0 0 0"/>
       <geometry>
-        <mesh filename="${body_mesh_file}" scale="${body_mesh_scale}"/>
+        <box size="${body_length} ${body_width} ${body_height}"/>
       </geometry>
-      <material name="gray"/>
+      <material name="body_gray"/>
     </visual>
     <collision>
-      <origin xyz="0 0 ${body_height/2.0 - wheel_radius}" rpy="0 0 0"/>
+      <origin xyz="0 0 ${body_height / 2.0 - drive_wheel_radius}" rpy="0 0 0"/>
       <geometry>
         <box size="${body_length} ${body_width} ${body_height}"/>
@@ -84,116 +74,50 @@
     </collision>
     <inertial>
-      <origin xyz="0 0 0" rpy="0 0 0"/>
+      <origin xyz="0 0 ${body_height / 2.0 - drive_wheel_radius}" rpy="0 0 0"/>
       <mass value="15.0"/>
-      <inertia ixx="0.5" ixy="0.0" ixz="0.0"
-               iyy="0.8" iyz="0.0"
-               izz="1.0"/>
+      <inertia ixx="0.5" ixy="0.0" ixz="0.0" iyy="0.8" iyz="0.0" izz="1.0"/>
     </inertial>
   </link>
-  <!-- ===================== -->
-  <!-- Left wheel            -->
-  <!-- ===================== -->
-  <link name="left_wheel_link">
-    <visual>
-      <origin xyz="0 0 0" rpy="0 ${pi/2} 0"/>
-      <geometry>
-        <cylinder radius="${wheel_radius}" length="${wheel_thickness}"/>
-      </geometry>
-      <material name="black"/>
-    </visual>
-    <collision>
-      <origin xyz="0 0 0" rpy="0 ${pi/2} 0"/>
-      <geometry>
-        <cylinder radius="${wheel_radius}" length="${wheel_thickness}"/>
-      </geometry>
-    </collision>
-    <inertial>
-      <origin xyz="0 0 0" rpy="0 0 0"/>
-      <mass value="1.0"/>
-      <inertia ixx="0.01" ixy="0.0" ixz="0.0"
-               iyy="0.01" iyz="0.0"
-               izz="0.01"/>
-    </inertial>
-  </link>
-  <joint name="left_wheel_joint" type="continuous">
-    <parent link="base_link"/>
-    <child link="left_wheel_link"/>
-    <origin xyz="0 ${wheel_separation/2.0} 0" rpy="0 0 0"/>
-    <axis xyz="0 1 0"/>
-  </joint>
-  <!-- ===================== -->
-  <!-- Right wheel           -->
-  <!-- ===================== -->
-  <link name="right_wheel_link">
-    <visual>
-      <origin xyz="0 0 0" rpy="0 ${pi/2} 0"/>
-      <geometry>
-        <cylinder radius="${wheel_radius}" length="${wheel_thickness}"/>
-      </geometry>
-      <material name="black"/>
-    </visual>
-    <collision>
-      <origin xyz="0 0 0" rpy="0 ${pi/2} 0"/>
-      <geometry>
-        <cylinder radius="${wheel_radius}" length="${wheel_thickness}"/>
-      </geometry>
-    </collision>
-    <inertial>
-      <origin xyz="0 0 0" rpy="0 0 0"/>
-      <mass value="1.0"/>
-      <inertia ixx="0.01" ixy="0.0" ixz="0.0"
-               iyy="0.01" iyz="0.0"
-               izz="0.01"/>
-    </inertial>
-  </link>
-  <joint name="right_wheel_joint" type="continuous">
-    <parent link="base_link"/>
-    <child link="right_wheel_link"/>
-    <origin xyz="0 ${-wheel_separation/2.0} 0" rpy="0 0 0"/>
-    <axis xyz="0 1 0"/>
-  </joint>
-  <!-- ===================== -->
-  <!-- Caster wheel          -->
-  <!-- ===================== -->
-  <link name="caster_wheel_link">
-    <visual>
-      <origin xyz="0 0 0" rpy="0 ${pi/2} 0"/>
-      <geometry>
-        <cylinder radius="${caster_radius}" length="${caster_thickness}"/>
-      </geometry>
-      <material name="black"/>
-    </visual>
-    <collision>
-      <origin xyz="0 0 0" rpy="0 ${pi/2} 0"/>
-      <geometry>
-        <cylinder radius="${caster_radius}" length="${caster_thickness}"/>
-      </geometry>
-    </collision>
-    <inertial>
-      <origin xyz="0 0 0" rpy="0 0 0"/>
-      <mass value="0.5"/>
-      <inertia ixx="0.003" ixy="0.0" ixz="0.0"
-               iyy="0.003" iyz="0.0"
-               izz="0.003"/>
-    </inertial>
-  </link>
-  <joint name="caster_wheel_joint" type="fixed">
-    <parent link="base_link"/>
-    <child link="caster_wheel_link"/>
-    <origin xyz="-0.30 0 ${-(wheel_radius - caster_radius)}" rpy="0 0 0"/>
-  </joint>
-  <!-- ===================== -->
-  <!-- LiDAR                 -->
-  <!-- ===================== -->
+  <xacro:macro name="drive_wheel" params="side y">
+    <link name="${side}_wheel_link">
+      <visual>
+        <origin xyz="0 0 0" rpy="${pi / 2.0} 0 0"/>
+        <geometry>
+          <cylinder radius="${drive_wheel_radius}" length="${drive_wheel_thickness}"/>
+        </geometry>
+        <material name="wheel_black"/>
+      </visual>
+      <collision>
+        <origin xyz="0 0 0" rpy="${pi / 2.0} 0 0"/>
+        <geometry>
+          <cylinder radius="${drive_wheel_radius}" length="${drive_wheel_thickness}"/>
+        </geometry>
+      </collision>
+      <inertial>
+        <origin xyz="0 0 0" rpy="0 0 0"/>
+        <mass value="1.0"/>
+        <inertia ixx="0.01" ixy="0.0" ixz="0.0" iyy="0.01" iyz="0.0" izz="0.01"/>
+      </inertial>
+    </link>
+    <joint name="${side}_wheel_joint" type="continuous">
+      <parent link="base_link"/>
+      <child link="${side}_wheel_link"/>
+      <origin xyz="0 ${y} 0" rpy="0 0 0"/>
+      <axis xyz="0 1 0"/>
+    </joint>
+  </xacro:macro>
+  <xacro:drive_wheel side="left" y="${wheel_separation / 2.0}"/>
+  <xacro:drive_wheel side="right" y="${-wheel_separation / 2.0}"/>
+  <!-- TODO: Add caster link and joint after caster wheel position is finalized. -->
   <link name="lidar_link">
     <visual>
       <geometry>
-        <box size="0.037 0.037 0.024"/>
+        <box size="${lidar_size}"/>
       </geometry>
-      <material name="blue"/>
+      <material name="lidar_blue"/>
     </visual>
     <collision>
       <geometry>
-        <box size="0.037 0.037 0.024"/>
+        <box size="${lidar_size}"/>
       </geometry>
     </collision>
@@ -204,17 +128,14 @@
     <origin xyz="${lidar_x} ${lidar_y} ${lidar_z}" rpy="0 0 0"/>
   </joint>
-  <!-- ===================== -->
-  <!-- IMU                   -->
-  <!-- ===================== -->
   <link name="imu_link">
     <visual>
       <geometry>
-        <box size="0.04 0.04 0.02"/>
+        <box size="${imu_size}"/>
       </geometry>
-      <material name="green"/>
+      <material name="imu_green"/>
     </visual>
     <collision>
       <geometry>
-        <box size="0.04 0.04 0.02"/>
+        <box size="${imu_size}"/>
       </geometry>
     </collision>
@@ -225,18 +146,22 @@
     <origin xyz="${imu_x} ${imu_y} ${imu_z}" rpy="0 0 0"/>
   </joint>
-  <!-- ===================== -->
-  <!-- ToF sensors           -->
-  <!-- ===================== -->
-  <xacro:macro name="tof_sensor" params="name px py pz yaw">
+  <xacro:macro name="tof_sensor" params="name x y z yaw">
     <link name="${name}">
       <visual>
         <geometry>
-          <box size="0.03 0.02 0.02"/>
+          <box size="${tof_size}"/>
         </geometry>
-        <material name="blue"/>
+        <material name="tof_orange"/>
+      </visual>
+      <visual>
+        <origin xyz="0.055 0 0" rpy="0 0 0"/>
+        <geometry>
+          <box size="${tof_direction_size}"/>
+        </geometry>
+        <material name="tof_direction_yellow"/>
       </visual>
       <collision>
         <geometry>
-          <box size="0.03 0.02 0.02"/>
+          <box size="${tof_size}"/>
         </geometry>
       </collision>
@@ -245,10 +170,30 @@
       <parent link="base_link"/>
       <child link="${name}"/>
-      <origin xyz="${px} ${py} ${pz}" rpy="0 0 ${yaw}"/>
+      <origin xyz="${x} ${y} ${z}" rpy="0 0 ${yaw}"/>
     </joint>
   </xacro:macro>
-  <xacro:tof_sensor name="tof_link_0" px="${tof0_x}" py="${tof0_y}" pz="${tof0_z}" yaw="0"/>
-  <xacro:tof_sensor name="tof_link_1" px="${tof1_x}" py="${tof1_y}" pz="${tof1_z}" yaw="0"/>
-  <xacro:tof_sensor name="tof_link_2" px="${tof2_x}" py="${tof2_y}" pz="${tof2_z}" yaw="${pi}"/>
-  <xacro:tof_sensor name="tof_link_3" px="${tof3_x}" py="${tof3_y}" pz="${tof3_z}" yaw="${pi}"/>
+  <xacro:tof_sensor
+    name="tof_front_left_link"
+    x="${tof_front_left_x}"
+    y="${tof_front_left_y}"
+    z="${tof_front_left_z}"
+    yaw="${tof_front_left_yaw}"/>
+  <xacro:tof_sensor
+    name="tof_front_right_link"
+    x="${tof_front_right_x}"
+    y="${tof_front_right_y}"
+    z="${tof_front_right_z}"
+    yaw="${tof_front_right_yaw}"/>
+  <xacro:tof_sensor
+    name="tof_rear_left_link"
+    x="${tof_rear_left_x}"
+    y="${tof_rear_left_y}"
+    z="${tof_rear_left_z}"
+    yaw="${tof_rear_left_yaw}"/>
+  <xacro:tof_sensor
+    name="tof_rear_right_link"
+    x="${tof_rear_right_x}"
+    y="${tof_rear_right_y}"
+    z="${tof_rear_right_z}"
+    yaw="${tof_rear_right_yaw}"/>
 </robot>

Commit message: [KMJ] feat: slam preparation

File: robot/description/urdf/robot.urdf.xacro (robot description, xacro)
@@ -110,5 +110,5 @@
   <xacro:drive_wheel side="right" y="${-wheel_separation / 2.0}"/>
   <!-- TODO: Add caster link and joint after caster wheel position is finalized. -->
-  <link name="lidar_link">
+  <link name="laser_frame">
     <visual>
       <geometry>
@@ -125,5 +125,5 @@
   <joint name="lidar_joint" type="fixed">
     <parent link="base_link"/>
-    <child link="lidar_link"/>
+    <child link="laser_frame"/>
     <origin xyz="${lidar_x} ${lidar_y} ${lidar_z}" rpy="0 0 0"/>
   </joint>

Commit message: [KMJ] feat: second slam prepreparations

File: robot/description/urdf/robot.urdf.xacro (robot description, xacro)
@@ -56,10 +56,10 @@
     <parent link="base_footprint"/>
     <child link="base_link"/>
-    <origin xyz="0 0 ${drive_wheel_radius}" rpy="0 0 0"/>
+    <origin xyz="0 0 ${drive_wheel_diameter}" rpy="0 0 0"/>
   </joint>
   <link name="base_link">
     <!-- TODO: Replace body primitive with Fusion 360 STL or DAE mesh after export. -->
     <visual>
-      <origin xyz="0 0 ${body_height / 2.0 - drive_wheel_radius}" rpy="0 0 0"/>
+      <origin xyz="0 0 0" rpy="0 0 0"/>
       <geometry>
         <box size="${body_length} ${body_width} ${body_height}"/>
@@ -68,5 +68,5 @@
     </visual>
     <collision>
-      <origin xyz="0 0 ${body_height / 2.0 - drive_wheel_radius}" rpy="0 0 0"/>
+      <origin xyz="0 0 0" rpy="0 0 0"/>
       <geometry>
         <box size="${body_length} ${body_width} ${body_height}"/>
@@ -74,5 +74,5 @@
     </collision>
     <inertial>
-      <origin xyz="0 0 ${body_height / 2.0 - drive_wheel_radius}" rpy="0 0 0"/>
+      <origin xyz="0 0 0" rpy="0 0 0"/>
       <mass value="15.0"/>
       <inertia ixx="0.5" ixy="0.0" ixz="0.0" iyy="0.8" iyz="0.0" izz="1.0"/>
@@ -103,5 +103,5 @@
       <parent link="base_link"/>
       <child link="${side}_wheel_link"/>
-      <origin xyz="0 ${y} 0" rpy="0 0 0"/>
+      <origin xyz="0 ${y} ${drive_wheel_radius - drive_wheel_diameter}" rpy="0 0 0"/>
       <axis xyz="0 1 0"/>
     </joint>

Commit message: [KMJ] refactor: add invalid reading logic to tof node

File: robot/description/urdf/robot.urdf.xacro (robot description, xacro)
@@ -21,9 +21,9 @@
   <xacro:property name="tof_front_left_y" value="0.32"/>
   <xacro:property name="tof_front_left_z" value="0.15"/>
-  <xacro:property name="tof_front_left_yaw" value="0.436332"/>
+  <xacro:property name="tof_front_left_yaw" value="2.007128"/>
   <xacro:property name="tof_front_right_x" value="0.22"/>
   <xacro:property name="tof_front_right_y" value="-0.32"/>
   <xacro:property name="tof_front_right_z" value="0.15"/>
-  <xacro:property name="tof_front_right_yaw" value="-0.436332"/>
+  <xacro:property name="tof_front_right_yaw" value="-2.007128"/>
   <xacro:property name="tof_rear_left_x" value="-0.55"/>
   <xacro:property name="tof_rear_left_y" value="0.28"/>

Commit message: [KMJ] refactor: ToF pipeline for async sensor reads and VL53L1X rear_center support

File: robot/description/urdf/robot.urdf.xacro (robot description, xacro)
@@ -34,4 +34,8 @@
   <xacro:property name="tof_rear_right_z" value="0.15"/>
   <xacro:property name="tof_rear_right_yaw" value="-2.70526"/>
+  <xacro:property name="tof_rear_center_x" value="-0.55"/>
+  <xacro:property name="tof_rear_center_y" value="0.0"/>
+  <xacro:property name="tof_rear_center_z" value="0.15"/>
+  <xacro:property name="tof_rear_center_yaw" value="3.141593"/>
   <material name="body_gray">
     <color rgba="0.55 0.58 0.62 1.0"/>
@@ -197,3 +201,9 @@
     z="${tof_rear_right_z}"
     yaw="${tof_rear_right_yaw}"/>
+  <xacro:tof_sensor
+    name="tof_rear_center_link"
+    x="${tof_rear_center_x}"
+    y="${tof_rear_center_y}"
+    z="${tof_rear_center_z}"
+    yaw="${tof_rear_center_yaw}"/>
 </robot>

Commit message: [KMJ] update: align robot dimensions, footprint, and sensor transforms

File: robot/description/urdf/robot.urdf.xacro (robot description, xacro)
@@ -1,8 +1,8 @@
 <?xml version="1.0"?>
 <robot name="hospital_delivery_robot" xmlns:xacro="http://www.ros.org/wiki/xacro">
-  <xacro:property name="body_length" value="0.8"/>
-  <xacro:property name="body_width" value="0.59"/>
-  <xacro:property name="body_height" value="0.19"/>
-  <xacro:property name="wheel_separation" value="0.38"/>
+  <xacro:property name="body_length" value="0.8182"/>
+  <xacro:property name="body_width" value="0.696"/>
+  <xacro:property name="body_height" value="0.9737"/>
+  <xacro:property name="wheel_separation" value="0.35"/>
   <xacro:property name="drive_wheel_diameter" value="0.125"/>
   <xacro:property name="drive_wheel_radius" value="0.0625"/>
@@ -15,23 +15,23 @@
   <xacro:property name="lidar_y" value="0.0"/>
   <xacro:property name="lidar_z" value="0.175"/>
-  <xacro:property name="imu_x" value="0.30"/>
-  <xacro:property name="imu_y" value="0.0"/>
-  <xacro:property name="imu_z" value="0.0"/>
+  <xacro:property name="imu_x" value="-0.07"/>
+  <xacro:property name="imu_y" value="0.01"/>
+  <xacro:property name="imu_z" value="0.015"/>
   <xacro:property name="tof_front_left_x" value="0.22"/>
-  <xacro:property name="tof_front_left_y" value="0.32"/>
+  <xacro:property name="tof_front_left_y" value="0.37"/>
   <xacro:property name="tof_front_left_z" value="0.15"/>
-  <xacro:property name="tof_front_left_yaw" value="2.007128"/>
+  <xacro:property name="tof_front_left_yaw" value="0.209440"/>
   <xacro:property name="tof_front_right_x" value="0.22"/>
-  <xacro:property name="tof_front_right_y" value="-0.32"/>
+  <xacro:property name="tof_front_right_y" value="-0.23"/>
   <xacro:property name="tof_front_right_z" value="0.15"/>
-  <xacro:property name="tof_front_right_yaw" value="-2.007128"/>
+  <xacro:property name="tof_front_right_yaw" value="-0.209440"/>
   <xacro:property name="tof_rear_left_x" value="-0.55"/>
-  <xacro:property name="tof_rear_left_y" value="0.28"/>
+  <xacro:property name="tof_rear_left_y" value="0.32"/>
   <xacro:property name="tof_rear_left_z" value="0.15"/>
-  <xacro:property name="tof_rear_left_yaw" value="2.70526"/>
+  <xacro:property name="tof_rear_left_yaw" value="2.932153"/>
   <xacro:property name="tof_rear_right_x" value="-0.55"/>
-  <xacro:property name="tof_rear_right_y" value="-0.28"/>
+  <xacro:property name="tof_rear_right_y" value="-0.23"/>
   <xacro:property name="tof_rear_right_z" value="0.15"/>
-  <xacro:property name="tof_rear_right_yaw" value="-2.70526"/>
+  <xacro:property name="tof_rear_right_yaw" value="-2.932153"/>
   <xacro:property name="tof_rear_center_x" value="-0.55"/>
   <xacro:property name="tof_rear_center_y" value="0.0"/>
