Commit message: [KMJ] fix: align lidar frame orientation in URDF

File: robot/description/urdf/robot.urdf.xacro (robot description, xacro)
@@ -130,5 +130,5 @@
     <parent link="base_link"/>
     <child link="laser_frame"/>
-    <origin xyz="${lidar_x} ${lidar_y} ${lidar_z}" rpy="0 0 0"/>
+    <origin xyz="${lidar_x} ${lidar_y} ${lidar_z}" rpy="0 0 ${pi}"/>
   </joint>
   <link name="imu_link">

Commit message: [KMJ] fix: update robot body dimensions and clearance

File: robot/description/urdf/robot.urdf.xacro (robot description, xacro)
@@ -1,7 +1,7 @@
 <?xml version="1.0"?>
 <robot name="hospital_delivery_robot" xmlns:xacro="http://www.ros.org/wiki/xacro">
-  <xacro:property name="body_length" value="0.8182"/>
-  <xacro:property name="body_width" value="0.696"/>
-  <xacro:property name="body_height" value="0.9737"/>
+  <xacro:property name="body_length" value="0.83"/>
+  <xacro:property name="body_width" value="0.71"/>
+  <xacro:property name="body_height" value="0.91"/>
   <xacro:property name="wheel_separation" value="0.35"/>
   <xacro:property name="drive_wheel_diameter" value="0.125"/>
@@ -65,5 +65,5 @@
     <!-- TODO: Replace body primitive with Fusion 360 STL or DAE mesh after export. -->
     <visual>
-      <origin xyz="0 0 0" rpy="0 0 0"/>
+      <origin xyz="0 0 0.43" rpy="0 0 0"/>
       <geometry>
         <box size="${body_length} ${body_width} ${body_height}"/>
@@ -72,5 +72,5 @@
     </visual>
     <collision>
-      <origin xyz="0 0 0" rpy="0 0 0"/>
+      <origin xyz="0 0 0.43" rpy="0 0 0"/>
       <geometry>
         <box size="${body_length} ${body_width} ${body_height}"/>
@@ -78,5 +78,5 @@
     </collision>
     <inertial>
-      <origin xyz="0 0 0" rpy="0 0 0"/>
+      <origin xyz="0 0 0.43" rpy="0 0 0"/>
       <mass value="15.0"/>
       <inertia ixx="0.5" ixy="0.0" ixz="0.0" iyy="0.8" iyz="0.0" izz="1.0"/>

Commit message: [KMJ] fix: correct body and sensor offset direction

File: robot/description/urdf/robot.urdf.xacro (robot description, xacro)
@@ -8,4 +8,5 @@
   <xacro:property name="drive_wheel_radius" value="0.0625"/>
   <xacro:property name="drive_wheel_thickness" value="0.04"/>
+  <xacro:property name="body_mount_shift_x" value="-0.16"/>
   <xacro:property name="lidar_size" value="0.037 0.037 0.024"/>
   <xacro:property name="imu_size" value="0.045 0.035 0.018"/>
@@ -15,6 +16,6 @@
   <xacro:property name="lidar_y" value="0.0"/>
   <xacro:property name="lidar_z" value="0.175"/>
-  <xacro:property name="imu_x" value="-0.07"/>
-  <xacro:property name="imu_y" value="0.01"/>
+  <xacro:property name="imu_x" value="0.0"/>
+  <xacro:property name="imu_y" value="0.0"/>
   <xacro:property name="imu_z" value="0.015"/>
   <xacro:property name="tof_front_left_x" value="0.22"/>
@@ -23,5 +24,5 @@
   <xacro:property name="tof_front_left_yaw" value="0.209440"/>
   <xacro:property name="tof_front_right_x" value="0.22"/>
-  <xacro:property name="tof_front_right_y" value="-0.23"/>
+  <xacro:property name="tof_front_right_y" value="-0.37"/>
   <xacro:property name="tof_front_right_z" value="0.15"/>
   <xacro:property name="tof_front_right_yaw" value="-0.209440"/>
@@ -31,8 +32,8 @@
   <xacro:property name="tof_rear_left_yaw" value="2.932153"/>
   <xacro:property name="tof_rear_right_x" value="-0.55"/>
-  <xacro:property name="tof_rear_right_y" value="-0.23"/>
+  <xacro:property name="tof_rear_right_y" value="-0.32"/>
   <xacro:property name="tof_rear_right_z" value="0.15"/>
   <xacro:property name="tof_rear_right_yaw" value="-2.932153"/>
-  <xacro:property name="tof_rear_center_x" value="-0.55"/>
+  <xacro:property name="tof_rear_center_x" value="-0.60"/>
   <xacro:property name="tof_rear_center_y" value="0.0"/>
   <xacro:property name="tof_rear_center_z" value="0.15"/>
@@ -65,5 +66,5 @@
     <!-- TODO: Replace body primitive with Fusion 360 STL or DAE mesh after export. -->
     <visual>
-      <origin xyz="0 0 0.43" rpy="0 0 0"/>
+      <origin xyz="${body_mount_shift_x} 0 0.43" rpy="0 0 0"/>
       <geometry>
         <box size="${body_length} ${body_width} ${body_height}"/>
@@ -72,5 +73,5 @@
     </visual>
     <collision>
-      <origin xyz="0 0 0.43" rpy="0 0 0"/>
+      <origin xyz="${body_mount_shift_x} 0 0.43" rpy="0 0 0"/>
       <geometry>
         <box size="${body_length} ${body_width} ${body_height}"/>
@@ -78,5 +79,5 @@
     </collision>
     <inertial>
-      <origin xyz="0 0 0.43" rpy="0 0 0"/>
+      <origin xyz="${body_mount_shift_x} 0 0.43" rpy="0 0 0"/>
       <mass value="15.0"/>
       <inertia ixx="0.5" ixy="0.0" ixz="0.0" iyy="0.8" iyz="0.0" izz="1.0"/>
